File: TET.kicad_pcb (KiCad board)
At the start: 4 copper layers, 90.2 x 95.9 mm, 67 parts, among them J1 SWT, M1 MountingHole, M2 MountingHole, M3 MountingHole, M4 MountingHole, U1 E80-900M2213S_C42464134, U10 TLV75533PDBVR, U11 INA226AIDGSR, U12 TCAN330GDCNR, U13 SMA-KWE_C7498154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

Commit message: ✨ feat(schematic): start connections for STM32L4
Parts:
- removed D1, D2, D3: SS14, Diode_SMD:D_SMA
- removed R1: 0.1, Resistor_SMD:R_0603_1608Metric
- removed R2, R3: 10k, Resistor_SMD:R_0603_1608Metric
- removed U10: TLV75533PDBVR, TET-Footprints:SOT-23-5_L3.0-W1.7-P0.95-LS2.8-BR
- removed U11: INA226AIDGSR, TET-Footprints:MSOP-10_L3.0-W3.0-P0.50-LS5.0-BL
- added C16: 100nF, Capacitor_SMD:C_0603_1608Metric, F.Cu at (136.1, 85.6)
- added C17: 100nF, Capacitor_SMD:C_0603_1608Metric, F.Cu at (140.1, 68.0)
- added C18: 100nF, Capacitor_SMD:C_0603_1608Metric, F.Cu at (140.1, 70.5)
- added C19: 100nF, Capacitor_SMD:C_0603_1608Metric, F.Cu at (140.1, 73.0)
- added C20: 10uF, Capacitor_SMD:C_0603_1608Metric, F.Cu at (140.1, 75.5)
- added C21: 10nF, Capacitor_SMD:C_0603_1608Metric, F.Cu at (140.1, 78.0)
- added C22: 1uF, Capacitor_SMD:C_0603_1608Metric, F.Cu at (140.1, 80.5)
- added C23: 1uF, Capacitor_SMD:C_0603_1608Metric, F.Cu at (140.1, 83.0)
- added C24: 0.1uF, Capacitor_SMD:C_0603_1608Metric, F.Cu at (102.4, 68.0)
- added C25: 22uF, Capacitor_SMD:C_0603_1608Metric, F.Cu at (102.4, 70.5)
- added C26: 22uF, Capacitor_SMD:C_0603_1608Metric, F.Cu at (102.4, 73.0)
- added D7: SS14, Diode_SMD:D_SMA, F.Cu at (104.5, 84.1)
- added D8: SS14, Diode_SMD:D_SMA, F.Cu at (104.5, 88.6)
- added D9: SS14, Diode_SMD:D_SMA, F.Cu at (104.5, 93.2)
- added FB1: 120R, Inductor_SMD:L_0603_1608Metric, F.Cu at (140.1, 85.6)
- added R19: 10k, Resistor_SMD:R_0603_1608Metric, F.Cu at (102.4, 75.5)
- added R20: 0.1, Resistor_SMD:R_0603_1608Metric, F.Cu at (102.4, 78.0)
- added R21: 10k, Resistor_SMD:R_0603_1608Metric, F.Cu at (102.4, 80.5)
- added U19: INA226AIDGSR, TET-Footprints:MSOP-10_L3.0-W3.0-P0.50-LS5.0-BL, F.Cu at (102.8, 98.9)
- added U20: TLV75533PDBVR, TET-Footprints:SOT-23-5_L3.0-W1.7-P0.95-LS2.8-BR, F.Cu at (102.7, 104.5)
- C1: value 22uF -> 100nF
- C2: value 22uF -> 20pF
- C3: value 0.1uF -> 20pF
- U13: value SMA-KWE_C7498154 -> SMA_1
- U14: value SMA-KWE_C7498154 -> SMA_2
- U15: value X50328MSB2GI -> 8 MHz
- moved R12 43.1 mm to (148.2, 68.0)
- moved R15 43.1 mm to (148.2, 75.5)
- moved R4 43.1 mm to (144.2, 68.0)
- moved R7 43.1 mm to (144.2, 75.5)
- moved R13 43.1 mm to (148.2, 70.5)
- moved R14 43.1 mm to (148.2, 73.0)
- moved R18 43.1 mm to (148.2, 78.0)
- moved R5 43.1 mm to (144.2, 70.5)
- moved R6 43.1 mm to (144.2, 73.0)
- moved R8 43.1 mm to (144.2, 78.0)
- moved R9 43.1 mm to (144.2, 80.5)
- moved C1 36.7 mm to (132.1, 68.0)
- moved C2 36.7 mm to (132.1, 70.5)
- moved C3 36.7 mm to (132.1, 73.0)
- moved C4 36.7 mm to (132.1, 75.5)
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Connections:
- C1 pad 1: +3.3V -> /NRST
- C2 pad 1: Net-(U10-IN) -> /OSC_IN
- C3 pad 1: +3.3V -> /OSC_OUT
- U15 pad 1: unconnected-(U15-OSC1-Pad1) -> /OSC_OUT
- U15 pad 2: unconnected-(U15-OSC2-Pad2) -> /OSC_IN
- U2 pad 1: unconnected-(U2-VBAT-Pad1) -> +3.3V
- U2 pad 11: /SCL0 -> unconnected-(U2-PA1-Pad11)
- U2 pad 12: /SDA0 -> unconnected-(U2-PA2-Pad12)
- U2 pad 23: unconnected-(U2-VSS-Pad23) -> GND
- U2 pad 24: unconnected-(U2-VDD-Pad24) -> +3.3V
- U2 pad 34: unconnected-(U2-PA13(JTMSSWDIO-Pad34) -> /SWDIO
- U2 pad 35: unconnected-(U2-VSS-Pad35) -> GND
- U2 pad 36: unconnected-(U2-VDD-Pad36) -> +3.3V
- U2 pad 37: unconnected-(U2-PA14(JTCKSWCLK)-Pad37) -> /SWCLK
- U2 pad 44: unconnected-(U2-PH3/BOOT0-Pad44) -> /BOOT0
- U2 pad 47: unconnected-(U2-VSS-Pad47) -> GND
- U2 pad 48: unconnected-(U2-VDD-Pad48) -> +3.3V
- U2 pad 5: unconnected-(U2-PH0-OSC_IN(PH0)-Pad5) -> /OSC_IN
- U2 pad 6: unconnected-(U2-PH1-OSC_OUT(PH1)-Pad6) -> /OSC_OUT
- U2 pad 7: unconnected-(U2-NRST-Pad7) -> /NRST
- U2 pad 8: unconnected-(U2-VSSA/VREF--Pad8) -> GND
- U2 pad 9: unconnected-(U2-VDDA/VREF+-Pad9) -> +3.3VA

Commit message: ♻️ ref(schematic): change MCU from 48 pins to 64 pins
Parts:
- added U10: STM32L431RBT6TR, TET-Footprints:LQFP-64_L10.0-W10.0-P0.50-LS12.0-BL, F.Cu at (91.2, 64.0)
Connections:
- U12 pad 1: /CAN_TXD -> /CAN1_TX
- U12 pad 4: /CAN_RXD -> /CAN1_RX
- U12 pad 8: /CAN_STB -> /CAN1_STB
- U2 pad 10: unconnected-(U2-PA0-Pad10) -> /FLASH1_CS
- U2 pad 11: unconnected-(U2-PA1-Pad11) -> /FLASH2_CS
- U2 pad 12: unconnected-(U2-PA2-Pad12) -> /FLASH3_CS
- U2 pad 13: unconnected-(U2-PA3-Pad13) -> /QSPI_CLK
- U2 pad 14: unconnected-(U2-PA4-Pad14) -> /RX_LED
- U2 pad 15: unconnected-(U2-PA5-Pad15) -> /TMP112_A_ALERT
- U2 pad 16: unconnected-(U2-PA6-Pad16) -> /TMP112_B_ALERT
- U2 pad 17: unconnected-(U2-PA7-Pad17) -> /TMP112_C_ALERT
- U2 pad 18: unconnected-(U2-PB0-Pad18) -> /QSPI_IO1
- U2 pad 19: unconnected-(U2-PB1-Pad19) -> /QSPI_IO0
- U2 pad 20: unconnected-(U2-PB2-Pad20) -> /TX_LED
- U2 pad 21: unconnected-(U2-PB10-Pad21) -> /USART3_TX
- U2 pad 22: unconnected-(U2-PB11-Pad22) -> /USART3_RX
- U2 pad 25: unconnected-(U2-PB12-Pad25) -> /LR_NSS
- U2 pad 26: unconnected-(U2-PB13-Pad26) -> /LR_BUSY
- U2 pad 27: unconnected-(U2-PB14-Pad27) -> /CAN1_STB
- U2 pad 28: unconnected-(U2-PB15-Pad28) -> INA226_ALERT
- U2 pad 29: unconnected-(U2-PA8-Pad29) -> /TMP112_D_ALERT
- U2 pad 30: unconnected-(U2-PA9-Pad30) -> /USART1_TX
- U2 pad 31: unconnected-(U2-PA10-Pad31) -> /USART1_RX
- U2 pad 32: unconnected-(U2-PA11-Pad32) -> /CAN1_TX
- U2 pad 33: unconnected-(U2-PA12-Pad33) -> /CAN1_RX
- U2 pad 39: unconnected-(U2-PB3(JTDOTRACESWO)-Pad39) -> /SPI1_SCK
- U2 pad 40: unconnected-(U2-PB4(NJTRST)-Pad40) -> /SPI1_MISO
- U2 pad 41: unconnected-(U2-PB5-Pad41) -> /SPI1_MOSI
- U2 pad 42: unconnected-(U2-PB6-Pad42) -> /QSPI_IO3
- U2 pad 43: unconnected-(U2-PB7-Pad43) -> /QSPI_IO2
- U2 pad 45: unconnected-(U2-PB8-Pad45) -> /I2C1_SCL
- U2 pad 46: unconnected-(U2-PB9-Pad46) -> /I2C1_SDA
- U6 pad 1: /SCL0 -> /I2C1_SCL
- U6 pad 4: /SCL0 -> /I2C1_SCL
- U6 pad 6: /SDA0 -> /I2C1_SDA
- U7 pad 1: /SCL0 -> /I2C1_SCL
- U7 pad 6: /SDA0 -> /I2C1_SDA
- U8 pad 1: /SCL0 -> /I2C1_SCL
- U8 pad 4: /SDA0 -> /I2C1_SDA
- U8 pad 6: /SDA0 -> /I2C1_SDA
- U9 pad 1: /SCL0 -> /I2C1_SCL
- U9 pad 6: /SDA0 -> /I2C1_SDA
