File: hardware/PCB/TET-Power-Supply.kicad_sch (KiCad schematic)
At the start: 24 parts, among them U10 TLV75533PDBVR, U6 5015, U7 5015, U8 INA226AQDGSRQ1, U9 TMP112AIDRLR

Commit message: feat(hardware): implement TET module PCB design and restructure project
Parts:
- removed U8: INA226AQDGSRQ1, TET-Footprints:VSSOP-10_L3.0-W3.0-P0.50-LS4.9-BL, symbol TET-Symbols:INA226AQDGSRQ1
- added U23: INA226AIDGSR, TET-Footprints:MSOP-10_L3.0-W3.0-P0.50-LS5.0-BL, symbol TET-Symbols:INA226AIDGSR
- C15, C16, C17, C18: footprint Capacitor_SMD:C_0603_1608Metric -> Capacitor_SMD:C_0402_1005Metric
- R19, R20, R21, R23, R24, R25: footprint Resistor_SMD:R_0603_1608Metric -> Resistor_SMD:R_0402_1005Metric
- R22: value 0.1 -> 2m; footprint Resistor_SMD:R_1206_3216Metric -> TET-Footprints:RES-SMD_L6.3-W3.1-1
Connections:
- net +3.3V: now also R19.2, U23.6 (VS+); no longer R19.1
- net +5V: now also U23.10 (VIN+), U23.8 (VBUS), U23.9 (VIN-)
- net GND: now also U23.1 (A1), U23.2 (A0), U23.7 (GND)
- net I2C1_SCL: now also U23.5 (SCL)
- net I2C1_SDA: now also U23.4 (SDA)
- net PWR_INA_ALERT: now also R19.1, U23.3 (Alert); no longer R19.2
- net PWR_1: now reaches H1.46 (Pin_46)
- net PWR_1: now also D1.2 (A)
- net PWR_2: now reaches H1.48 (Pin_48)
- net PWR_2: now also D2.2 (A)
- net PWR_3: now reaches H1.50 (Pin_50)
- net PWR_3: now also D3.2 (A)
- net CAN_A_H renamed CAN_A_N
- net CAN_A_L renamed CAN_A_P
- net PWR_4: no longer names the net of H1.52 (Pin_52)
- net PWR_4: no longer D1.2 (A)
- net PWR_5: no longer names the net of H2.34 (Pin_34)
- net PWR_5: no longer D2.2 (A)
- net PWR_6: no longer names the net of H2.36 (Pin_36)
- net PWR_6: no longer D3.2 (A)
- net TMP_A_ALERT renamed TMP_B_ALERT
- net UART_A_RX: no longer names the net of H1.7 (Pin_7)
- net UART_A_TX: no longer names the net of H1.5 (Pin_5)
- net UART_B_RX: no longer names the net of H1.8 (Pin_8)
- net UART_B_TX: no longer names the net of H1.6 (Pin_6)
- no-connect marks 90 -> 94
Other:
- note added: "CAN_H"
- note added: "CAN_L"
- moved on the sheet: R19

Commit message: feat(hardware): complete PCB layout and project structure
Parts:
- C2: renamed from C15; value 0.1uF -> 100nF
- C3: renamed from C16; footprint Capacitor_SMD:C_0402_1005Metric -> Capacitor_SMD:C_0805_2012Metric
- C4: renamed from C17; footprint Capacitor_SMD:C_0402_1005Metric -> Capacitor_SMD:C_0805_2012Metric
- C5: renamed from C18; value 0.1uF -> 100nF
- H1, H2: now not fitted; now left out of the parts list
- R7: renamed from R22; LCSC (none) -> C695817
- renumbered R19 to R1, R25 to R10, R20 to R2, R21 to R5, R23 to R8, R24 to R9, U6 to U1, U7 to U2, U23 to U3, U9 to U6, U10 to U7
Connections:
- net +5V: no longer C3.1, R7.2, R9.1, U3.8 (VBUS), U3.9 (VIN-), U7.1 (IN)
- new net SYS_LOAD: C3.1, R7.2, R9.1, U3.8 (VBUS), U3.9 (VIN-), U7.1 (IN)
Other:
- moved on the sheet: C3

Commit message: feat(hardware): release v1r2
Parts:
- removed C3, C4: 22uF, Capacitor_SMD:C_0805_2012Metric, symbol Device:C_Small
- removed D1, D2, D3: SS14, Diode_SMD:D_SMA, symbol Device:D_Schottky_Small
- removed R9: 10k, Resistor_SMD:R_0402_1005Metric, symbol Device:R_Small
- removed U7: TLV75533PDBVR, TET-Footprints:SOT-23-5_L3.0-W1.7-P0.95-LS2.8-BR, symbol TET-Symbols:TLV75533PDBVR
Connections:
- net PWR_1 is gone; now on net PWR: H1.46 (Pin_46)
- net PWR_2 is gone; now on net PWR: H1.48 (Pin_48)
- net PWR_3 is gone; now on net PWR: H1.50 (Pin_50)
- net SYS_LOAD is gone; now on net +3.3V: R7.2, U3.8 (VBUS), U3.9 (VIN-)
- net +5V renamed PWR
- no-connect marks 94 -> 93
Other:
- note added: "PWR_1"
- note added: "PWR_2"
- note added: "PWR_3"
- note removed: "5 V enters from the EPS (PWR_4-6), passes through a current/voltage monitor (INA226), and is regulated to 3.3 V by an LDO (TLV755)."
- note removed: "CHANNEL AGREGATOR DIODES"
- note removed: "LDO 3.3 V"
