File: hardware/PCB/TET.kicad_pcb (KiCad board)
At the start: 4 copper layers, 90.2 x 95.9 mm, 94 parts, among them J1 SWD, U10 TLV75533PDBVR, U11 SMA_1, U12 W25Q128JVSIQTR, U13 W25Q128JVSIQTR, U14 E80-900M2213S, U15 SMA_2, U16 W25Q128JVSIQTR, U17 TMP112AIDRLR, U19 TMP112AIDRLR, U20 STM32L431CCT6, U21 INA226AIDGSR, U23 INA226AIDGSR, U4 TMP112AIDRLR, U5 TCAN3414DR, U6 5015, U7 5015, U8 8 MHz, U9 TMP112AIDRLR

Commit message: feat(hardware): complete PCB layout and project structure
Parts:
- removed the G*** at (103.5, 134.2)
- added G***: LOGO, TET-Footprints:LibreCube_logo_22.4mm, F.Cu at (103.0, 134.4)
- C1, C14, C26, C27: value 0.1uF -> 100nF
- C2: renamed from C15; value 0.1uF -> 100nF
- C21, C29, C34: footprint Capacitor_SMD:C_0402_1005Metric -> Capacitor_SMD:C_0805_2012Metric
- C3: renamed from C16; footprint Capacitor_SMD:C_0402_1005Metric -> Capacitor_SMD:C_0805_2012Metric
- C4: renamed from C17; footprint Capacitor_SMD:C_0402_1005Metric -> Capacitor_SMD:C_0805_2012Metric
- C5: renamed from C18; value 0.1uF -> 100nF
- R3, R4: value 60 -> 60.4
- U11: value SMA_1 -> SMA
- U15: value SMA_2 -> SMA
- moved REF1 75.9 mm to (166.6, 56.9)
- moved D6 4.09 mm to (99.7, 99.2)
- moved D4 4.09 mm to (108.5, 99.2)
- moved D5 4.09 mm to (104.1, 99.2)
- moved R10 4.09 mm to (99.3, 97.3)
- moved R2 4.09 mm to (108.0, 97.3)
- moved R5 4.09 mm to (103.7, 97.3)
- moved G*** 3.50 mm to (153.1, 132.2)
- moved C34 2.20 mm to (128.8, 63.3)
- moved R9 1.96 mm to (159.5, 77.2), turned to 180 degrees
- moved J1 1.00 mm to (89.2, 82.9)
- moved C4 0.59 mm to (152.9, 79.3)
- moved C29 0.50 mm to (97.8, 69.8)
- moved C3 0.40 mm to (159.5, 79.8)
- moved C21 0.30 mm to (140.8, 97.5)
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- renumbered R19 to R1, R25 to R10, R20 to R2, R21 to R5, R22 to R7, R23 to R8, R24 to R9, U6 to U1, U7 to U2, U23 to U3, U9 to U6, U10 to U7
Connections:
- C21 pad 1: +3.3V -> /RF_Transceiver/RF_LOAD
- C22 pad 1: +3.3V -> /RF_Transceiver/RF_LOAD
- C3 pad 1: +5V -> /Power_Supply/SYS_LOAD
- R28 pad 1: +3.3V -> /RF_Transceiver/RF_LOAD
- R32 pad 1: +3.3V -> /RF_Transceiver/RF_LOAD
- R7 pad 2: +5V -> /Power_Supply/SYS_LOAD
- R9 pad 1: +5V -> /Power_Supply/SYS_LOAD
- U14 pad 25: +3.3V -> /RF_Transceiver/RF_LOAD
- U21 pad 10: +3.3V -> /RF_Transceiver/RF_LOAD
- U3 pad 8: +5V -> /Power_Supply/SYS_LOAD
- U3 pad 9: +5V -> /Power_Supply/SYS_LOAD
- U7 pad 1: +5V -> /Power_Supply/SYS_LOAD
Routing:
- net /RF_Transceiver/RF_LOAD: track 0.00 -> 33.3 mm
- net /Power_Supply/SYS_LOAD: track 0.00 -> 25.7 mm
- net +5V: track 92.7 -> 69.4 mm
- net +3.3V: track 127.0 -> 107.4 mm
- net GND: track 108.5 -> 116.4 mm, vias 104 -> 106
- net /RX_LED: track 41.0 -> 36.6 mm
- net /TX_LED: track 38.8 -> 35.5 mm
- net /RF_INA_ALERT: track 55.8 -> 53.9 mm
- net /SWDIO: track 75.4 -> 74.2 mm
- net Net-(U7-EN): track 3.00 -> 1.98 mm
- net /SWCLK: track 73.1 -> 72.1 mm
- net /NRST: track 75.2 -> 74.2 mm
- net /SWO: track 74.4 -> 73.5 mm
- net /I2C1_SCL: track 69.2 -> 70.0 mm
- net /I2C2_SCL: track 71.2 -> 72.1 mm
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- added copper zone on B.Cu, net GND
Other:
- board text added: "2.4 GHz"
- board text added: "3.3V"
- board text added: "5V IN"
- board text added: "CAN TERM."
- board text added: "CH1"
- board text added: "CH2"
- board text added: "CH3"
- board text added: "CLK"
- board text added: "DIO"
- board text added: "GND"
- board text added: "GND IN"
- board text added: "MEM 1"
- board text added: "NRST"
- board text added: "Part No.: 1eb0b9ce Version: v1r1 Designed by: Rodrigo A."
- board text added: "SWO"
- board text added: "Sub GHz"
- board text added: "TET Module Telemetry, Encoding & Transmission"
- board text removed: "Telemetry, Encoding & Transmission (TET) Module - V1.0"

Commit message: feat(hardware): release v1r2
Parts:
- removed C3, C4: 22uF, Capacitor_SMD:C_0805_2012Metric
- removed D1, D2, D3: SS14, Diode_SMD:D_SMA
- removed R9: 10k, Resistor_SMD:R_0402_1005Metric
- removed U7: TLV75533PDBVR, TET-Footprints:SOT-23-5_L3.0-W1.7-P0.95-LS2.8-BR
- moved C5 23.2 mm to (141.7, 66.7), turned to 90 degrees
- moved U6 19.9 mm to (144.0, 67.0), turned to 0 degrees
- moved R8 18.7 mm to (146.2, 65.0), turned to -90 degrees
- moved C2 6.32 mm to (155.4, 70.7)
- moved R1 6.32 mm to (146.8, 69.9)
- moved R7 6.32 mm to (159.9, 69.2)
- moved U3 6.32 mm to (151.5, 69.9)
- moved U2 4.00 mm to (159.7, 107.6)
Connections:
- H1 pad 46: /Power_Supply/PWR_1 -> /Power_Supply/PWR
- H1 pad 48: /Power_Supply/PWR_2 -> /Power_Supply/PWR
- H1 pad 50: /Power_Supply/PWR_3 -> /Power_Supply/PWR
- R7 pad 1: +5V -> /Power_Supply/PWR
- R7 pad 2: /Power_Supply/SYS_LOAD -> +3.3V
- U1 pad 1: +5V -> /Power_Supply/PWR
- U3 pad 10: +5V -> /Power_Supply/PWR
- U3 pad 8: /Power_Supply/SYS_LOAD -> +3.3V
- U3 pad 9: /Power_Supply/SYS_LOAD -> +3.3V
Routing:
- net +5V: track 69.4 -> 0.00 mm
- net /Power_Supply/PWR: track 0.00 -> 57.6 mm, vias 0 -> 9
- net /I2C1_SDA: track 74.9 -> 48.3 mm
- net /Power_Supply/SYS_LOAD: track 25.7 -> 0.00 mm
- net /I2C1_SCL: track 70.0 -> 47.1 mm, vias 6 -> 5
- net +3.3V: track 107.4 -> 120.9 mm, vias 32 -> 40
- net /TMP_B_ALERT: track 37.5 -> 25.1 mm
- net /Power_Supply/PWR_2: track 9.90 -> 0.00 mm
- net /Power_Supply/PWR_3: track 9.77 -> 0.00 mm
- net /Power_Supply/PWR_1: track 9.74 -> 0.00 mm
- net /PWR_INA_ALERT: track 30.3 -> 25.3 mm
- net GND: track 116.4 -> 120.1 mm, vias 106 -> 98
- net /SPI1_MISO: track 51.9 -> 48.7 mm
- net /SPI1_MOSI: track 41.3 -> 38.1 mm
- net Net-(U7-EN): track 1.98 -> 0.00 mm
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- added copper zone on In2.Cu, net /Power_Supply/PWR
Other:
- board text added: "3.3V IN"
- board text added: "Part No.: f2defc5c Version: v1r2 Designed by: Rodrigo A."
- board text removed: "5V IN"
- board text removed: "CH1"
- board text removed: "CH2"
- board text removed: "CH3"
- board text removed: "Part No.: 1eb0b9ce Version: v1r1 Designed by: Rodrigo A."
